File: g2g_kicad/G2g.sch (KiCad schematic (older format))
At the start: 12 parts, among them U1 NANOPI, U2 mux

Commit message: Increase heiht
Parts:
- U1: symbol nanopi:nanopi -> G2g-rescue:nanopi-nanopi
- U2: symbol nanopi:mux -> G2g-rescue:mux-nanopi
Changed lines of the file:
@@
 	4550 3850 4800 3850
 $Comp
-L nanopi:nanopi U1
+L G2g-rescue:nanopi-nanopi U1
 U 1 1 5C711050
 P 5150 3250
@@
 	4450 4050 4650 4050
 $Comp
-L nanopi:mux U2
+L G2g-rescue:mux-nanopi U2
 U 1 1 5C71D95E
 P 4850 6300

Commit message: Add Nut bolt holes
Parts:
- U1: footprint myLib:PinHeader_1x16_P2.54mm_Vertical -> myLib:nanopi_duo
- U2: footprint myLib:1x12 -> myLib:tca9548a
Changed lines of the file:
@@
 F 0 "U1" H 5150 4015 50  0000 C CNN
 F 1 "NANOPI" H 5150 3924 50  0000 C CNN
-F 2 "myLib:PinHeader_1x16_P2.54mm_Vertical" H 5150 3950 50  0001 C CNN
+F 2 "myLib:nanopi_duo" H 5150 3950 50  0001 C CNN
 F 3 "" H 5150 3950 50  0001 C CNN
 	1    5150 3250
@@
 F 0 "U2" H 4825 6925 50  0000 C CNN
 F 1 "mux" H 4825 6834 50  0000 C CNN
-F 2 "myLib:1x12" H 4850 6850 50  0001 C CNN
+F 2 "myLib:tca9548a" H 4850 6850 50  0001 C CNN
 F 3 "" H 4850 6850 50  0001 C CNN
 	1    4850 6300
